File: hardware/DesktopClock.kicad_sch (KiCad schematic)
At the start: 37 parts, among them J1 USB_C_Receptacle_USB2.0_16P, J2 Conn_01x14, J3 Conn_01x02, SW1 SW_SPST, SW2 SW_SPST, U1 BMI270, U2 USBLC6-2SC6, U3 LM1117LD-3.3, U4 BME688, U5 ESP32-S3-WROOM-1

Commit message: schem ver1.0
Connections:
- net BUZZER: now also U5.16 (IO46)
Changed lines of the file:
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@@
+	(wire
+		(pts
+			(xy 238.76 92.71) (xy 254 92.71)
+		)
+		(stroke
+			(width 0)
+			(type default)
+		)
+	)
 	(wire
 		(pts
@@
 		)
 	)
+	(label "BUZZER"
+		(at 240.03 92.71 0)
+		(effects
+			(font
+				(size 1.27 1.27)
+			)
+			(justify left bottom)
+		)
+	)

Commit message: rev 3.0
Parts:
- removed BZ1: Buzzer, symbol Device:Buzzer
- added D5: 1N5819WS, Diode_SMD:D_SOD-323, symbol Diode:1N5819WS
- added LS1: CSS-0575A-SMT, CSS-0575A-SMT:CUI_CSS-0575A-SMT, symbol CSS-0575A-SMT:CSS-0575A-SMT
- added Q1: BC847, Package_TO_SOT_SMD:SOT-23_Handsoldering, symbol Transistor_BJT:BC847
- added R10: 180, Resistor_SMD:R_0603_1608Metric_Pad0.98x0.95mm_HandSolder, symbol Device:R_Small
- C1, C2, C3, C4, C5, C6, C7, C8, C9: footprint (none) -> Capacitor_SMD:C_0603_1608Metric_Pad1.08x0.95mm_HandSolder
- D2: footprint (none) -> LED_SMD:LED_0805_2012Metric_Pad1.15x1.40mm_HandSolder
- H1, H2, H3, H4: footprint (none) -> MountingHole:MountingHole_3.2mm_M3; now in the parts list
- J1: footprint (none) -> Connector_USB:USB_C_Receptacle_GCT_USB4105-xx-A_16P_TopMnt_Horizontal
- J2: footprint (none) -> Connector_FFC-FPC:Amphenol_F32Q-1A7x1-11014_1x14-1MP_P0.5mm_Horizontal
- J3: footprint (none) -> Connector_PinHeader_2.54mm:PinHeader_1x02_P2.54mm_Horizontal
- R1, R2, R3, R4, R5, R6, R7, R8, R9: footprint (none) -> Resistor_SMD:R_0603_1608Metric_Pad0.98x0.95mm_HandSolder
- SW1, SW2: footprint (none) -> Button_Switch_SMD:SW_SPST_B3U-1000P
Connections:
- net +3.3V: now also D5.1 (K), LS1.1
- net BUZZER: now also R10.1
- net GND: now also Q1.2 (E)
- new net: D5.2 (A), LS1.2, Q1.3 (C)
- new net: Q1.1 (B), R10.2
- no-connect marks 10 -> 25

Commit message: Layout complete
Parts:
- removed U3: LM1117LD-3.3, Package_SON:WSON-8-1EP_4x4mm_P0.8mm_EP2.2x3mm, symbol Regulator_Linear:LM1117LD-3.3
- added U3: LM1117MP-3.3, Package_TO_SOT_SMD:SOT-223-3_TabPin2, symbol Regulator_Linear:LM1117MP-3.3
- SW1: value SW_SPST -> RST
- SW2: value SW_SPST -> BOOT
Connections:
- net +3.3V: now also U3.2 (VO)
- net +5V: now also U3.3 (VI)
- net GND: now also U3.1 (GND)
- net INT2: now reaches U5.26 (IO45)
- net INT2: now also U1.9 (INT2)
- net INT1: now reaches U5.35 (IO42)
- net INT1: now also U1.4 (INT1)
- no-connect marks 25 -> 27
